File: ByteBridge.kicad_sch (KiCad schematic)
At the start: 23 parts, among them J1 USB_C_Receptacle_USB2.0_16P, J2 Conn_01x04_Pin, J5 Conn_01x03_Pin, U1 AMS1117-3.3, U2 CP2102N-Axx-xQFN28

Commit message: fix: spelling
Parts:
- R4: Manufacturer (none) -> YAGEO; Manufcturer YAGEO -> (none)
- R5: Manufacturer (none) -> YAGEO; Manufaturer YAGEO -> (none)
Changed lines of the file:
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@@
 			)
 		)
-		(property "Manufcturer" "YAGEO"
+		(property "Manufacturer" "YAGEO"
 			(at 97.79 76.2 90)
 			(effects
@@
 			)
 		)
-		(property "Manufaturer" "YAGEO"
+		(property "Manufacturer" "YAGEO"
 			(at 105.41 81.28 90)
 			(effects
